Commit message: Fix scan_joint on burger model

File: turtlebot3_description/urdf/turtlebot3_burger.urdf.xacro (robot description, xacro)
@@ -116,5 +116,5 @@
     <parent link="base_link"/>
     <child link="base_scan"/>
-    <origin xyz="-0.032 0 0.172" rpy="0 0 0"/>
+    <origin xyz="-0.039 0 0.172" rpy="0 0 0"/>
   </joint>
   <link name="base_scan">
